Commit message: Update fastbot_body.xacro

File: fastbot/fastbot_description/models/urdf/fastbot_body.xacro (robot description, xacro)
@@ -16,5 +16,5 @@
             <origin xyz="0.0573343 -0.0691426 0.00134516" rpy="0 -0 3.14159"/>
             <geometry>
-                <mesh filename="file:///ros2_ws/src/fastbot/fastbot_description/onshape/assets/fastbot_chassis.stl"/>
+                <mesh filename="$(find-pkg-share fastbot_description)/onshape/assets/fastbot_chassis.stl"/>
             </geometry>
             <material name="fastbot_chassis_material">
@@ -26,5 +26,5 @@
             <!--<origin xyz="0.0 0.0 -0.00134516" rpy="0 0 0"/>-->
             <geometry>
-                <mesh filename="file:///ros2_ws/src/fastbot/fastbot_description/onshape/assets/fastbot_chassis.stl"/>
+                <mesh filename="$(find-pkg-share fastbot_description)/onshape/assets/fastbot_chassis.stl"/>
                 <!--<box size="0.12 0.155 0.115" />-->
             </geometry>
@@ -42,5 +42,5 @@
             <origin xyz="0.0935 -0.00775 -0.036" rpy="-1.5708 -1.5708 0"/>
             <geometry>
-                <mesh filename="file:///ros2_ws/src/fastbot/fastbot_description/onshape/assets/fastbot_motor.stl"/>
+                <mesh filename="$(find-pkg-share fastbot_description)/onshape/assets/fastbot_motor.stl"/>
             </geometry>
             <material name="fastbot_motor_material">
@@ -51,5 +51,5 @@
             <origin xyz="0.0935 -0.00775 -0.036" rpy="-1.5708 -1.5708 0"/>
             <geometry>
-                <mesh filename="file:///ros2_ws/src/fastbot/fastbot_description/onshape/assets/fastbot_motor.stl"/>
+                <mesh filename="$(find-pkg-share fastbot_description)/onshape/assets/fastbot_motor.stl"/>
             </geometry>
         </collision>
@@ -66,5 +66,5 @@
             <origin xyz="0.1135 0.0162 0.103475" rpy="1.5708 1.5708 0"/>
             <geometry>
-                <mesh filename="file:///ros2_ws/src/fastbot/fastbot_description/onshape/assets/wheel_d65x25_v1.stl"/>
+                <mesh filename="$(find-pkg-share fastbot_description)/onshape/assets/wheel_d65x25_v1.stl"/>
             </geometry>
             <material name="wheel_d65x25_v1_material">
@@ -75,5 +75,5 @@
             <origin xyz="0.1135 0.0162 0.103475" rpy="1.5708 1.5708 0"/>
             <geometry>
-                <mesh filename="file:///ros2_ws/src/fastbot/fastbot_description/onshape/assets/wheel_d65x25_v1.stl"/>
+                <mesh filename="$(find-pkg-share fastbot_description)/onshape/assets/wheel_d65x25_v1.stl"/>
             </geometry>
         </collision>
@@ -82,5 +82,5 @@
             <origin xyz="0.1135 0.0162 0.1039" rpy="1.5708 1.5708 0"/>
             <geometry>
-                <mesh filename="file:///ros2_ws/src/fastbot/fastbot_description/onshape/assets/wheel_d65x25_v1__2.stl"/>
+                <mesh filename="$(find-pkg-share fastbot_description)/onshape/assets/wheel_d65x25_v1__2.stl"/>
             </geometry>
             <material name="wheel_d65x25_v1_2_material">
@@ -91,5 +91,5 @@
             <origin xyz="0.1135 0.0162 0.1039" rpy="1.5708 1.5708 0"/>
             <geometry>
-                <mesh filename="file:///ros2_ws/src/fastbot/fastbot_description/onshape/assets/wheel_d65x25_v1__2.stl"/>
+                <mesh filename="$(find-pkg-share fastbot_description)/onshape/assets/wheel_d65x25_v1__2.stl"/>
             </geometry>
         </collision>
@@ -120,5 +120,5 @@
             <origin xyz="0.0935 -0.02475 -0.036" rpy="-1.5708 -1.5708 0"/>
             <geometry>
-                <mesh filename="file:///ros2_ws/src/fastbot/fastbot_description/onshape/assets/fastbot_motor.stl"/>
+                <mesh filename="$(find-pkg-share fastbot_description)/onshape/assets/fastbot_motor.stl"/>
             </geometry>
             <material name="fastbot_motor_2_material">
@@ -129,5 +129,5 @@
             <origin xyz="0.0935 -0.02475 -0.036" rpy="-1.5708 -1.5708 0"/>
             <geometry>
-                <mesh filename="file:///ros2_ws/src/fastbot/fastbot_description/onshape/assets/fastbot_motor.stl"/>
+                <mesh filename="$(find-pkg-share fastbot_description)/onshape/assets/fastbot_motor.stl"/>
             </geometry>
         </collision>
@@ -144,5 +144,5 @@
             <origin xyz="0.1135 0.0162 0.1039" rpy="1.5708 1.5708 0"/>
             <geometry>
-                <mesh filename="file:///ros2_ws/src/fastbot/fastbot_description/onshape/assets/wheel_d65x25_v1__2.stl"/>
+                <mesh filename="$(find-pkg-share fastbot_description)/onshape/assets/wheel_d65x25_v1__2.stl"/>
             </geometry>
             <material name="wheel_d65x25_v1_3_material">
@@ -153,5 +153,5 @@
             <origin xyz="0.1135 0.0162 0.1039" rpy="1.5708 1.5708 0"/>
             <geometry>
-                <mesh filename="file:///ros2_ws/src/fastbot/fastbot_description/onshape/assets/wheel_d65x25_v1__2.stl"/>
+                <mesh filename="$(find-pkg-share fastbot_description)/onshape/assets/wheel_d65x25_v1__2.stl"/>
             </geometry>
         </collision>
@@ -160,5 +160,5 @@
             <origin xyz="0.1135 0.0162 0.104325" rpy="1.5708 1.5708 0"/>
             <geometry>
-                <mesh filename="file:///ros2_ws/src/fastbot/fastbot_description/onshape/assets/wheel_d65x25_v1.stl"/>
+                <mesh filename="$(find-pkg-share fastbot_description)/onshape/assets/wheel_d65x25_v1.stl"/>
             </geometry>
             <material name="wheel_d65x25_v1_4_material">
@@ -169,5 +169,5 @@
             <origin xyz="0.1135 0.0162 0.104325" rpy="1.5708 1.5708 0"/>
             <geometry>
-                <mesh filename="file:///ros2_ws/src/fastbot/fastbot_description/onshape/assets/wheel_d65x25_v1.stl"/>
+                <mesh filename="$(find-pkg-share fastbot_description)/onshape/assets/wheel_d65x25_v1.stl"/>
             </geometry>
         </collision>
@@ -198,5 +198,5 @@
             <origin xyz="-0.074 -0.06 0.11" rpy="-3.14159 5.94511e-32 -8.90522e-65"/>
             <geometry>
-                <mesh filename="file:///ros2_ws/src/fastbot/fastbot_description/onshape/assets/lslidar_n10.stl"/>
+                <mesh filename="$(find-pkg-share fastbot_description)/onshape/assets/lslidar_n10.stl"/>
             </geometry>
             <material name="lslidar_n10_material">
@@ -207,5 +207,5 @@
             <origin xyz="-0.074 -0.06 0.11" rpy="-3.14159 5.94511e-32 -8.90522e-65"/>
             <geometry>
-                <mesh filename="file:///ros2_ws/src/fastbot/fastbot_description/onshape/assets/lslidar_n10.stl"/>
+                <mesh filename="$(find-pkg-share fastbot_description)/onshape/assets/lslidar_n10.stl"/>
             </geometry>
         </collision>
@@ -229,5 +229,5 @@
             <origin xyz="-0.0105 0.0125 -0.00212" rpy="3.14159 -3.05067e-31 -1.55575e-61"/>
             <geometry>
-                <mesh filename="file:///ros2_ws/src/fastbot/fastbot_description/onshape/assets/raspicam.stl"/>
+                <mesh filename="$(find-pkg-share fastbot_description)/onshape/assets/raspicam.stl"/>
             </geometry>
             <material name="raspicam_material">
@@ -238,5 +238,5 @@
             <origin xyz="-0.0105 0.0125 -0.00212" rpy="3.14159 -3.05067e-31 -1.55575e-61"/>
             <geometry>
-                <mesh filename="file:///ros2_ws/src/fastbot/fastbot_description/onshape/assets/raspicam.stl"/>
+                <mesh filename="$(find-pkg-share fastbot_description)/onshape/assets/raspicam.stl"/>
             </geometry>
         </collision>
@@ -259,5 +259,5 @@
             <origin xyz="0.006731 0 -0.0106945" rpy="-1.5708 -0 0"/>
             <geometry>
-                <mesh filename="file:///ros2_ws/src/fastbot/fastbot_description/onshape/assets/pololu_ball_caster.stl"/>
+                <mesh filename="$(find-pkg-share fastbot_description)/onshape/assets/pololu_ball_caster.stl"/>
             </geometry>
             <material name="pololu_ball_caster_material">
@@ -268,5 +268,5 @@
             <origin xyz="0.006731 0 -0.0106945" rpy="-1.5708 -0 0"/>
             <geometry>
-                <mesh filename="file:///ros2_ws/src/fastbot/fastbot_description/onshape/assets/pololu_ball_caster.stl"/>
+                <mesh filename="$(find-pkg-share fastbot_description)/onshape/assets/pololu_ball_caster.stl"/>
             </geometry>
         </collision>

Commit message: Update fastbot_body.xacro

File: fastbot/fastbot_description/models/urdf/fastbot_body.xacro (robot description, xacro)
@@ -16,5 +16,5 @@
             <origin xyz="0.0573343 -0.0691426 0.00134516" rpy="0 -0 3.14159"/>
             <geometry>
-                <mesh filename="$(find-pkg-share fastbot_description)/onshape/assets/fastbot_chassis.stl"/>
+                <mesh filename="file:///ros2_ws/src/fastbot/fastbot_description/onshape/assets/fastbot_chassis.stl"/>
             </geometry>
             <material name="fastbot_chassis_material">
@@ -26,5 +26,5 @@
             <!--<origin xyz="0.0 0.0 -0.00134516" rpy="0 0 0"/>-->
             <geometry>
-                <mesh filename="$(find-pkg-share fastbot_description)/onshape/assets/fastbot_chassis.stl"/>
+                <mesh filename="file:///ros2_ws/src/fastbot/fastbot_description/onshape/assets/fastbot_chassis.stl"/>
                 <!--<box size="0.12 0.155 0.115" />-->
             </geometry>
@@ -42,5 +42,5 @@
             <origin xyz="0.0935 -0.00775 -0.036" rpy="-1.5708 -1.5708 0"/>
             <geometry>
-                <mesh filename="$(find-pkg-share fastbot_description)/onshape/assets/fastbot_motor.stl"/>
+                <mesh filename="file:///ros2_ws/src/fastbot/fastbot_description/onshape/assets/fastbot_motor.stl"/>
             </geometry>
             <material name="fastbot_motor_material">
@@ -51,5 +51,5 @@
             <origin xyz="0.0935 -0.00775 -0.036" rpy="-1.5708 -1.5708 0"/>
             <geometry>
-                <mesh filename="$(find-pkg-share fastbot_description)/onshape/assets/fastbot_motor.stl"/>
+                <mesh filename="file:///ros2_ws/src/fastbot/fastbot_description/onshape/assets/fastbot_motor.stl"/>
             </geometry>
         </collision>
@@ -66,5 +66,5 @@
             <origin xyz="0.1135 0.0162 0.103475" rpy="1.5708 1.5708 0"/>
             <geometry>
-                <mesh filename="$(find-pkg-share fastbot_description)/onshape/assets/wheel_d65x25_v1.stl"/>
+                <mesh filename="file:///ros2_ws/src/fastbot/fastbot_description/onshape/assets/wheel_d65x25_v1.stl"/>
             </geometry>
             <material name="wheel_d65x25_v1_material">
@@ -75,5 +75,5 @@
             <origin xyz="0.1135 0.0162 0.103475" rpy="1.5708 1.5708 0"/>
             <geometry>
-                <mesh filename="$(find-pkg-share fastbot_description)/onshape/assets/wheel_d65x25_v1.stl"/>
+                <mesh filename="file:///ros2_ws/src/fastbot/fastbot_description/onshape/assets/wheel_d65x25_v1.stl"/>
             </geometry>
         </collision>
@@ -82,5 +82,5 @@
             <origin xyz="0.1135 0.0162 0.1039" rpy="1.5708 1.5708 0"/>
             <geometry>
-                <mesh filename="$(find-pkg-share fastbot_description)/onshape/assets/wheel_d65x25_v1__2.stl"/>
+                <mesh filename="file:///ros2_ws/src/fastbot/fastbot_description/onshape/assets/wheel_d65x25_v1__2.stl"/>
             </geometry>
             <material name="wheel_d65x25_v1_2_material">
@@ -91,5 +91,5 @@
             <origin xyz="0.1135 0.0162 0.1039" rpy="1.5708 1.5708 0"/>
             <geometry>
-                <mesh filename="$(find-pkg-share fastbot_description)/onshape/assets/wheel_d65x25_v1__2.stl"/>
+                <mesh filename="file:///ros2_ws/src/fastbot/fastbot_description/onshape/assets/wheel_d65x25_v1__2.stl"/>
             </geometry>
         </collision>
@@ -120,5 +120,5 @@
             <origin xyz="0.0935 -0.02475 -0.036" rpy="-1.5708 -1.5708 0"/>
             <geometry>
-                <mesh filename="$(find-pkg-share fastbot_description)/onshape/assets/fastbot_motor.stl"/>
+                <mesh filename="file:///ros2_ws/src/fastbot/fastbot_description/onshape/assets/fastbot_motor.stl"/>
             </geometry>
             <material name="fastbot_motor_2_material">
@@ -129,5 +129,5 @@
             <origin xyz="0.0935 -0.02475 -0.036" rpy="-1.5708 -1.5708 0"/>
             <geometry>
-                <mesh filename="$(find-pkg-share fastbot_description)/onshape/assets/fastbot_motor.stl"/>
+                <mesh filename="file:///ros2_ws/src/fastbot/fastbot_description/onshape/assets/fastbot_motor.stl"/>
             </geometry>
         </collision>
@@ -144,5 +144,5 @@
             <origin xyz="0.1135 0.0162 0.1039" rpy="1.5708 1.5708 0"/>
             <geometry>
-                <mesh filename="$(find-pkg-share fastbot_description)/onshape/assets/wheel_d65x25_v1__2.stl"/>
+                <mesh filename="file:///ros2_ws/src/fastbot/fastbot_description/onshape/assets/wheel_d65x25_v1__2.stl"/>
             </geometry>
             <material name="wheel_d65x25_v1_3_material">
@@ -153,5 +153,5 @@
             <origin xyz="0.1135 0.0162 0.1039" rpy="1.5708 1.5708 0"/>
             <geometry>
-                <mesh filename="$(find-pkg-share fastbot_description)/onshape/assets/wheel_d65x25_v1__2.stl"/>
+                <mesh filename="file:///ros2_ws/src/fastbot/fastbot_description/onshape/assets/wheel_d65x25_v1__2.stl"/>
             </geometry>
         </collision>
@@ -160,5 +160,5 @@
             <origin xyz="0.1135 0.0162 0.104325" rpy="1.5708 1.5708 0"/>
             <geometry>
-                <mesh filename="$(find-pkg-share fastbot_description)/onshape/assets/wheel_d65x25_v1.stl"/>
+                <mesh filename="file:///ros2_ws/src/fastbot/fastbot_description/onshape/assets/wheel_d65x25_v1.stl"/>
             </geometry>
             <material name="wheel_d65x25_v1_4_material">
@@ -169,5 +169,5 @@
             <origin xyz="0.1135 0.0162 0.104325" rpy="1.5708 1.5708 0"/>
             <geometry>
-                <mesh filename="$(find-pkg-share fastbot_description)/onshape/assets/wheel_d65x25_v1.stl"/>
+                <mesh filename="file:///ros2_ws/src/fastbot/fastbot_description/onshape/assets/wheel_d65x25_v1.stl"/>
             </geometry>
         </collision>
@@ -198,5 +198,5 @@
             <origin xyz="-0.074 -0.06 0.11" rpy="-3.14159 5.94511e-32 -8.90522e-65"/>
             <geometry>
-                <mesh filename="$(find-pkg-share fastbot_description)/onshape/assets/lslidar_n10.stl"/>
+                <mesh filename="file:///ros2_ws/src/fastbot/fastbot_description/onshape/assets/lslidar_n10.stl"/>
             </geometry>
             <material name="lslidar_n10_material">
@@ -207,5 +207,5 @@
             <origin xyz="-0.074 -0.06 0.11" rpy="-3.14159 5.94511e-32 -8.90522e-65"/>
             <geometry>
-                <mesh filename="$(find-pkg-share fastbot_description)/onshape/assets/lslidar_n10.stl"/>
+                <mesh filename="file:///ros2_ws/src/fastbot/fastbot_description/onshape/assets/lslidar_n10.stl"/>
             </geometry>
         </collision>
@@ -229,5 +229,5 @@
             <origin xyz="-0.0105 0.0125 -0.00212" rpy="3.14159 -3.05067e-31 -1.55575e-61"/>
             <geometry>
-                <mesh filename="$(find-pkg-share fastbot_description)/onshape/assets/raspicam.stl"/>
+                <mesh filename="file:///ros2_ws/src/fastbot/fastbot_description/onshape/assets/raspicam.stl"/>
             </geometry>
             <material name="raspicam_material">
@@ -238,5 +238,5 @@
             <origin xyz="-0.0105 0.0125 -0.00212" rpy="3.14159 -3.05067e-31 -1.55575e-61"/>
             <geometry>
-                <mesh filename="$(find-pkg-share fastbot_description)/onshape/assets/raspicam.stl"/>
+                <mesh filename="file:///ros2_ws/src/fastbot/fastbot_description/onshape/assets/raspicam.stl"/>
             </geometry>
         </collision>
@@ -259,5 +259,5 @@
             <origin xyz="0.006731 0 -0.0106945" rpy="-1.5708 -0 0"/>
             <geometry>
-                <mesh filename="$(find-pkg-share fastbot_description)/onshape/assets/pololu_ball_caster.stl"/>
+                <mesh filename="file:///ros2_ws/src/fastbot/fastbot_description/onshape/assets/pololu_ball_caster.stl"/>
             </geometry>
             <material name="pololu_ball_caster_material">
@@ -268,5 +268,5 @@
             <origin xyz="0.006731 0 -0.0106945" rpy="-1.5708 -0 0"/>
             <geometry>
-                <mesh filename="$(find-pkg-share fastbot_description)/onshape/assets/pololu_ball_caster.stl"/>
+                <mesh filename="file:///ros2_ws/src/fastbot/fastbot_description/onshape/assets/pololu_ball_caster.stl"/>
             </geometry>
         </collision>
