Commit message: Update fastbot.xacro

File: fastbot/fastbot_description/models/urdf/fastbot.xacro (robot description, xacro)
@@ -16,5 +16,5 @@
             <origin xyz="0.06 -0.0698336 -0.002" rpy="0 -0 3.14159"/>
             <geometry>
-                <mesh filename="package://fastbot_description/onshape/assets/fastbot_chassis.stl"/>
+                <mesh filename="file://fastbot_description/onshape/assets/fastbot_chassis.stl"/>
             </geometry>
             <material name="base_link_material">
@@ -25,5 +25,5 @@
             <origin xyz="0.06 -0.0698336 -0.002" rpy="0 -0 3.14159"/>
             <geometry>
-                <mesh filename="package://fastbot_description/onshape/assets/fastbot_chassis.stl"/>
+                <mesh filename="file://fastbot_description/onshape/assets/fastbot_chassis.stl"/>
             </geometry>
         </collision>
@@ -40,5 +40,5 @@
             <origin xyz="0.0935 -0.00775 -0.036" rpy="-1.5708 -1.5708 0"/>
             <geometry>
-                <mesh filename="package://fastbot_description/onshape/assets/fastbot_motor.stl"/>
+                <mesh filename="file://fastbot_description/onshape/assets/fastbot_motor.stl"/>
             </geometry>
             <material name="fastbot_motor_material">
@@ -49,5 +49,5 @@
             <origin xyz="0.0935 -0.00775 -0.036" rpy="-1.5708 -1.5708 0"/>
             <geometry>
-                <mesh filename="package://fastbot_description/onshape/assets/fastbot_motor.stl"/>
+                <mesh filename="file://fastbot_description/onshape/assets/fastbot_motor.stl"/>
             </geometry>
         </collision>
@@ -64,5 +64,5 @@
             <origin xyz="0.1135 0.0162 0.103475" rpy="1.5708 1.5708 0"/>
             <geometry>
-                <mesh filename="package://fastbot_description/onshape/assets/wheel_d65x25_v1.stl"/>
+                <mesh filename="file://fastbot_description/onshape/assets/wheel_d65x25_v1.stl"/>
             </geometry>
             <material name="wheel_right_material">
@@ -73,5 +73,5 @@
             <origin xyz="0.1135 0.0162 0.103475" rpy="1.5708 1.5708 0"/>
             <geometry>
-                <mesh filename="package://fastbot_description/onshape/assets/wheel_d65x25_v1.stl"/>
+                <mesh filename="file://fastbot_description/onshape/assets/wheel_d65x25_v1.stl"/>
             </geometry>
         </collision>
@@ -80,5 +80,5 @@
             <origin xyz="0.1135 0.0162 0.1039" rpy="1.5708 1.5708 0"/>
             <geometry>
-                <mesh filename="package://fastbot_description/onshape/assets/wheel_d65x25_v1__2.stl"/>
+                <mesh filename="file://fastbot_description/onshape/assets/wheel_d65x25_v1__2.stl"/>
             </geometry>
             <material name="wheel_left_material">
@@ -89,5 +89,5 @@
             <origin xyz="0.1135 0.0162 0.1039" rpy="1.5708 1.5708 0"/>
             <geometry>
-                <mesh filename="package://fastbot_description/onshape/assets/wheel_d65x25_v1__2.stl"/>
+                <mesh filename="file://fastbot_description/onshape/assets/wheel_d65x25_v1__2.stl"/>
             </geometry>
         </collision>
@@ -120,5 +120,5 @@
             <origin xyz="0.0935 -0.02475 -0.036" rpy="-1.5708 -1.5708 0"/>
             <geometry>
-                <mesh filename="package://fastbot_description/onshape/assets/fastbot_motor.stl"/>
+                <mesh filename="file://fastbot_description/onshape/assets/fastbot_motor.stl"/>
             </geometry>
             <material name="fastbot_motor_2_material">
@@ -129,5 +129,5 @@
             <origin xyz="0.0935 -0.02475 -0.036" rpy="-1.5708 -1.5708 0"/>
             <geometry>
-                <mesh filename="package://fastbot_description/onshape/assets/fastbot_motor.stl"/>
+                <mesh filename="file://fastbot_description/onshape/assets/fastbot_motor.stl"/>
             </geometry>
         </collision>
@@ -144,5 +144,5 @@
             <origin xyz="0.1135 0.0162 0.1039" rpy="1.5708 1.5708 0"/>
             <geometry>
-                <mesh filename="package://fastbot_description/onshape/assets/wheel_d65x25_v1__2.stl"/>
+                <mesh filename="file://fastbot_description/onshape/assets/wheel_d65x25_v1__2.stl"/>
             </geometry>
             <material name="wheel_d65x25_v1_3_material">
@@ -153,5 +153,5 @@
             <origin xyz="0.1135 0.0162 0.1039" rpy="1.5708 1.5708 0"/>
             <geometry>
-                <mesh filename="package://fastbot_description/onshape/assets/wheel_d65x25_v1__2.stl"/>
+                <mesh filename="file://fastbot_description/onshape/assets/wheel_d65x25_v1__2.stl"/>
             </geometry>
         </collision>
@@ -160,5 +160,5 @@
             <origin xyz="0.1135 0.0162 0.104325" rpy="1.5708 1.5708 0"/>
             <geometry>
-                <mesh filename="package://fastbot_description/onshape/assets/wheel_d65x25_v1.stl"/>
+                <mesh filename="file://fastbot_description/onshape/assets/wheel_d65x25_v1.stl"/>
             </geometry>
             <material name="wheel_d65x25_v1_4_material">
@@ -169,5 +169,5 @@
             <origin xyz="0.1135 0.0162 0.104325" rpy="1.5708 1.5708 0"/>
             <geometry>
-                <mesh filename="package://fastbot_description/onshape/assets/wheel_d65x25_v1.stl"/>
+                <mesh filename="file://fastbot_description/onshape/assets/wheel_d65x25_v1.stl"/>
             </geometry>
         </collision>
@@ -200,5 +200,5 @@
             <origin xyz="-0.074 -0.06 0.11" rpy="-3.14159 5.94511e-32 -8.90522e-65"/>
             <geometry>
-                <mesh filename="package://fastbot_description/onshape/assets/n10_v2.stl"/>
+                <mesh filename="file://fastbot_description/onshape/assets/n10_v2.stl"/>
             </geometry>
             <material name="n10_v2_material">
@@ -209,5 +209,5 @@
             <origin xyz="-0.074 -0.06 0.11" rpy="-3.14159 5.94511e-32 -8.90522e-65"/>
             <geometry>
-                <mesh filename="package://fastbot_description/onshape/assets/n10_v2.stl"/>
+                <mesh filename="file://fastbot_description/onshape/assets/n10_v2.stl"/>
             </geometry>
         </collision>
@@ -232,5 +232,5 @@
             <origin xyz="-0.0105 0.0125 -0.00212" rpy="3.14159 -3.05067e-31 -1.55575e-61"/>
             <geometry>
-                <mesh filename="package://fastbot_description/onshape/assets/part_33.stl"/>
+                <mesh filename="file://fastbot_description/onshape/assets/part_33.stl"/>
             </geometry>
             <material name="camera_material">
@@ -241,5 +241,5 @@
             <origin xyz="-0.0105 0.0125 -0.00212" rpy="3.14159 -3.05067e-31 -1.55575e-61"/>
             <geometry>
-                <mesh filename="package://fastbot_description/onshape/assets/part_33.stl"/>
+                <mesh filename="file://fastbot_description/onshape/assets/part_33.stl"/>
             </geometry>
         </collision>

Commit message: Update fastbot.xacro

File: fastbot/fastbot_description/models/urdf/fastbot.xacro (robot description, xacro)
@@ -16,5 +16,5 @@
             <origin xyz="0.06 -0.0698336 -0.002" rpy="0 -0 3.14159"/>
             <geometry>
-                <mesh filename="file://fastbot_description/onshape/assets/fastbot_chassis.stl"/>
+                <mesh filename="file:///ros2_ws/src/fastbot/fastbot_description/onshape/assets/fastbot_chassis.stl"/>
             </geometry>
             <material name="base_link_material">
@@ -25,5 +25,5 @@
             <origin xyz="0.06 -0.0698336 -0.002" rpy="0 -0 3.14159"/>
             <geometry>
-                <mesh filename="file://fastbot_description/onshape/assets/fastbot_chassis.stl"/>
+                <mesh filename="file:///ros2_ws/src/fastbot/fastbot_description/onshape/assets/fastbot_chassis.stl"/>
             </geometry>
         </collision>
@@ -40,5 +40,5 @@
             <origin xyz="0.0935 -0.00775 -0.036" rpy="-1.5708 -1.5708 0"/>
             <geometry>
-                <mesh filename="file://fastbot_description/onshape/assets/fastbot_motor.stl"/>
+                <mesh filename="file:///ros2_ws/src/fastbot/fastbot_description/onshape/assets/fastbot_motor.stl"/>
             </geometry>
             <material name="fastbot_motor_material">
@@ -49,5 +49,5 @@
             <origin xyz="0.0935 -0.00775 -0.036" rpy="-1.5708 -1.5708 0"/>
             <geometry>
-                <mesh filename="file://fastbot_description/onshape/assets/fastbot_motor.stl"/>
+                <mesh filename="file:///ros2_ws/src/fastbot/fastbot_description/onshape/assets/fastbot_motor.stl"/>
             </geometry>
         </collision>
@@ -64,5 +64,5 @@
             <origin xyz="0.1135 0.0162 0.103475" rpy="1.5708 1.5708 0"/>
             <geometry>
-                <mesh filename="file://fastbot_description/onshape/assets/wheel_d65x25_v1.stl"/>
+                <mesh filename="file:///ros2_ws/src/fastbot/fastbot_description/onshape/assets/wheel_d65x25_v1.stl"/>
             </geometry>
             <material name="wheel_right_material">
@@ -73,5 +73,5 @@
             <origin xyz="0.1135 0.0162 0.103475" rpy="1.5708 1.5708 0"/>
             <geometry>
-                <mesh filename="file://fastbot_description/onshape/assets/wheel_d65x25_v1.stl"/>
+                <mesh filename="file:///ros2_ws/src/fastbot/fastbot_description/onshape/assets/wheel_d65x25_v1.stl"/>
             </geometry>
         </collision>
@@ -80,5 +80,5 @@
             <origin xyz="0.1135 0.0162 0.1039" rpy="1.5708 1.5708 0"/>
             <geometry>
-                <mesh filename="file://fastbot_description/onshape/assets/wheel_d65x25_v1__2.stl"/>
+                <mesh filename="file:///ros2_ws/src/fastbot/fastbot_description/onshape/assets/wheel_d65x25_v1__2.stl"/>
             </geometry>
             <material name="wheel_left_material">
@@ -89,5 +89,5 @@
             <origin xyz="0.1135 0.0162 0.1039" rpy="1.5708 1.5708 0"/>
             <geometry>
-                <mesh filename="file://fastbot_description/onshape/assets/wheel_d65x25_v1__2.stl"/>
+                <mesh filename="file:///ros2_ws/src/fastbot/fastbot_description/onshape/assets/wheel_d65x25_v1__2.stl"/>
             </geometry>
         </collision>
@@ -120,5 +120,5 @@
             <origin xyz="0.0935 -0.02475 -0.036" rpy="-1.5708 -1.5708 0"/>
             <geometry>
-                <mesh filename="file://fastbot_description/onshape/assets/fastbot_motor.stl"/>
+                <mesh filename="file:///ros2_ws/src/fastbot/fastbot_description/onshape/assets/fastbot_motor.stl"/>
             </geometry>
             <material name="fastbot_motor_2_material">
@@ -129,5 +129,5 @@
             <origin xyz="0.0935 -0.02475 -0.036" rpy="-1.5708 -1.5708 0"/>
             <geometry>
-                <mesh filename="file://fastbot_description/onshape/assets/fastbot_motor.stl"/>
+                <mesh filename="file:///ros2_ws/src/fastbot/fastbot_description/onshape/assets/fastbot_motor.stl"/>
             </geometry>
         </collision>
@@ -144,5 +144,5 @@
             <origin xyz="0.1135 0.0162 0.1039" rpy="1.5708 1.5708 0"/>
             <geometry>
-                <mesh filename="file://fastbot_description/onshape/assets/wheel_d65x25_v1__2.stl"/>
+                <mesh filename="file:///ros2_ws/src/fastbot/fastbot_description/onshape/assets/wheel_d65x25_v1__2.stl"/>
             </geometry>
             <material name="wheel_d65x25_v1_3_material">
@@ -153,5 +153,5 @@
             <origin xyz="0.1135 0.0162 0.1039" rpy="1.5708 1.5708 0"/>
             <geometry>
-                <mesh filename="file://fastbot_description/onshape/assets/wheel_d65x25_v1__2.stl"/>
+                <mesh filename="file:///ros2_ws/src/fastbot/fastbot_description/onshape/assets/wheel_d65x25_v1__2.stl"/>
             </geometry>
         </collision>
@@ -160,5 +160,5 @@
             <origin xyz="0.1135 0.0162 0.104325" rpy="1.5708 1.5708 0"/>
             <geometry>
-                <mesh filename="file://fastbot_description/onshape/assets/wheel_d65x25_v1.stl"/>
+                <mesh filename="file:///ros2_ws/src/fastbot/fastbot_description/onshape/assets/wheel_d65x25_v1.stl"/>
             </geometry>
             <material name="wheel_d65x25_v1_4_material">
@@ -169,5 +169,5 @@
             <origin xyz="0.1135 0.0162 0.104325" rpy="1.5708 1.5708 0"/>
             <geometry>
-                <mesh filename="file://fastbot_description/onshape/assets/wheel_d65x25_v1.stl"/>
+                <mesh filename="file:///ros2_ws/src/fastbot/fastbot_description/onshape/assets/wheel_d65x25_v1.stl"/>
             </geometry>
         </collision>
@@ -200,5 +200,5 @@
             <origin xyz="-0.074 -0.06 0.11" rpy="-3.14159 5.94511e-32 -8.90522e-65"/>
             <geometry>
-                <mesh filename="file://fastbot_description/onshape/assets/n10_v2.stl"/>
+                <mesh filename="file:///ros2_ws/src/fastbot/fastbot_description/onshape/assets/n10_v2.stl"/>
             </geometry>
             <material name="n10_v2_material">
@@ -209,5 +209,5 @@
             <origin xyz="-0.074 -0.06 0.11" rpy="-3.14159 5.94511e-32 -8.90522e-65"/>
             <geometry>
-                <mesh filename="file://fastbot_description/onshape/assets/n10_v2.stl"/>
+                <mesh filename="file:///ros2_ws/src/fastbot/fastbot_description/onshape/assets/n10_v2.stl"/>
             </geometry>
         </collision>
@@ -232,5 +232,5 @@
             <origin xyz="-0.0105 0.0125 -0.00212" rpy="3.14159 -3.05067e-31 -1.55575e-61"/>
             <geometry>
-                <mesh filename="file://fastbot_description/onshape/assets/part_33.stl"/>
+                <mesh filename="file:///ros2_ws/src/fastbot/fastbot_description/onshape/assets/part_33.stl"/>
             </geometry>
             <material name="camera_material">
@@ -241,5 +241,5 @@
             <origin xyz="-0.0105 0.0125 -0.00212" rpy="3.14159 -3.05067e-31 -1.55575e-61"/>
             <geometry>
-                <mesh filename="file://fastbot_description/onshape/assets/part_33.stl"/>
+                <mesh filename="file:///ros2_ws/src/fastbot/fastbot_description/onshape/assets/part_33.stl"/>
             </geometry>
         </collision>

Commit message: Update fastbot.xacro

File: fastbot/fastbot_description/models/urdf/fastbot.xacro (robot description, xacro)
@@ -16,5 +16,5 @@
             <origin xyz="0.06 -0.0698336 -0.002" rpy="0 -0 3.14159"/>
             <geometry>
-                <mesh filename="file:///ros2_ws/src/fastbot/fastbot_description/onshape/assets/fastbot_chassis.stl"/>
+                <mesh filename="$(find-pkg-share fastbot_description)/onshape/assets/fastbot_chassis.stl"/>
             </geometry>
             <material name="base_link_material">
@@ -25,5 +25,5 @@
             <origin xyz="0.06 -0.0698336 -0.002" rpy="0 -0 3.14159"/>
             <geometry>
-                <mesh filename="file:///ros2_ws/src/fastbot/fastbot_description/onshape/assets/fastbot_chassis.stl"/>
+                <mesh filename="$(find-pkg-share fastbot_description)/onshape/assets/fastbot_chassis.stl"/>
             </geometry>
         </collision>
@@ -40,5 +40,5 @@
             <origin xyz="0.0935 -0.00775 -0.036" rpy="-1.5708 -1.5708 0"/>
             <geometry>
-                <mesh filename="file:///ros2_ws/src/fastbot/fastbot_description/onshape/assets/fastbot_motor.stl"/>
+                <mesh filename="$(find-pkg-share fastbot_description)/onshape/assets/fastbot_motor.stl"/>
             </geometry>
             <material name="fastbot_motor_material">
@@ -49,5 +49,5 @@
             <origin xyz="0.0935 -0.00775 -0.036" rpy="-1.5708 -1.5708 0"/>
             <geometry>
-                <mesh filename="file:///ros2_ws/src/fastbot/fastbot_description/onshape/assets/fastbot_motor.stl"/>
+                <mesh filename="$(find-pkg-share fastbot_description)/onshape/assets/fastbot_motor.stl"/>
             </geometry>
         </collision>
@@ -64,5 +64,5 @@
             <origin xyz="0.1135 0.0162 0.103475" rpy="1.5708 1.5708 0"/>
             <geometry>
-                <mesh filename="file:///ros2_ws/src/fastbot/fastbot_description/onshape/assets/wheel_d65x25_v1.stl"/>
+                <mesh filename="$(find-pkg-share fastbot_description)/onshape/assets/wheel_d65x25_v1.stl"/>
             </geometry>
             <material name="wheel_right_material">
@@ -73,5 +73,5 @@
             <origin xyz="0.1135 0.0162 0.103475" rpy="1.5708 1.5708 0"/>
             <geometry>
-                <mesh filename="file:///ros2_ws/src/fastbot/fastbot_description/onshape/assets/wheel_d65x25_v1.stl"/>
+                <mesh filename="$(find-pkg-share fastbot_description)/onshape/assets/wheel_d65x25_v1.stl"/>
             </geometry>
         </collision>
@@ -80,5 +80,5 @@
             <origin xyz="0.1135 0.0162 0.1039" rpy="1.5708 1.5708 0"/>
             <geometry>
-                <mesh filename="file:///ros2_ws/src/fastbot/fastbot_description/onshape/assets/wheel_d65x25_v1__2.stl"/>
+                <mesh filename="$(find-pkg-share fastbot_description)/onshape/assets/wheel_d65x25_v1__2.stl"/>
             </geometry>
             <material name="wheel_left_material">
@@ -89,5 +89,5 @@
             <origin xyz="0.1135 0.0162 0.1039" rpy="1.5708 1.5708 0"/>
             <geometry>
-                <mesh filename="file:///ros2_ws/src/fastbot/fastbot_description/onshape/assets/wheel_d65x25_v1__2.stl"/>
+                <mesh filename="$(find-pkg-share fastbot_description)/onshape/assets/wheel_d65x25_v1__2.stl"/>
             </geometry>
         </collision>
@@ -120,5 +120,5 @@
             <origin xyz="0.0935 -0.02475 -0.036" rpy="-1.5708 -1.5708 0"/>
             <geometry>
-                <mesh filename="file:///ros2_ws/src/fastbot/fastbot_description/onshape/assets/fastbot_motor.stl"/>
+                <mesh filename="$(find-pkg-share fastbot_description)/onshape/assets/fastbot_motor.stl"/>
             </geometry>
             <material name="fastbot_motor_2_material">
@@ -129,5 +129,5 @@
             <origin xyz="0.0935 -0.02475 -0.036" rpy="-1.5708 -1.5708 0"/>
             <geometry>
-                <mesh filename="file:///ros2_ws/src/fastbot/fastbot_description/onshape/assets/fastbot_motor.stl"/>
+                <mesh filename="$(find-pkg-share fastbot_description)/onshape/assets/fastbot_motor.stl"/>
             </geometry>
         </collision>
@@ -144,5 +144,5 @@
             <origin xyz="0.1135 0.0162 0.1039" rpy="1.5708 1.5708 0"/>
             <geometry>
-                <mesh filename="file:///ros2_ws/src/fastbot/fastbot_description/onshape/assets/wheel_d65x25_v1__2.stl"/>
+                <mesh filename="$(find-pkg-share fastbot_description)/onshape/assets/wheel_d65x25_v1__2.stl"/>
             </geometry>
             <material name="wheel_d65x25_v1_3_material">
@@ -153,5 +153,5 @@
             <origin xyz="0.1135 0.0162 0.1039" rpy="1.5708 1.5708 0"/>
             <geometry>
-                <mesh filename="file:///ros2_ws/src/fastbot/fastbot_description/onshape/assets/wheel_d65x25_v1__2.stl"/>
+                <mesh filename="$(find-pkg-share fastbot_description)/onshape/assets/wheel_d65x25_v1__2.stl"/>
             </geometry>
         </collision>
@@ -160,5 +160,5 @@
             <origin xyz="0.1135 0.0162 0.104325" rpy="1.5708 1.5708 0"/>
             <geometry>
-                <mesh filename="file:///ros2_ws/src/fastbot/fastbot_description/onshape/assets/wheel_d65x25_v1.stl"/>
+                <mesh filename="$(find-pkg-share fastbot_description)/onshape/assets/wheel_d65x25_v1.stl"/>
             </geometry>
             <material name="wheel_d65x25_v1_4_material">
@@ -169,5 +169,5 @@
             <origin xyz="0.1135 0.0162 0.104325" rpy="1.5708 1.5708 0"/>
             <geometry>
-                <mesh filename="file:///ros2_ws/src/fastbot/fastbot_description/onshape/assets/wheel_d65x25_v1.stl"/>
+                <mesh filename="$(find-pkg-share fastbot_description)/onshape/assets/wheel_d65x25_v1.stl"/>
             </geometry>
         </collision>
@@ -200,5 +200,5 @@
             <origin xyz="-0.074 -0.06 0.11" rpy="-3.14159 5.94511e-32 -8.90522e-65"/>
             <geometry>
-                <mesh filename="file:///ros2_ws/src/fastbot/fastbot_description/onshape/assets/n10_v2.stl"/>
+                <mesh filename="$(find-pkg-share fastbot_description)/onshape/assets/n10_v2.stl"/>
             </geometry>
             <material name="n10_v2_material">
@@ -209,5 +209,5 @@
             <origin xyz="-0.074 -0.06 0.11" rpy="-3.14159 5.94511e-32 -8.90522e-65"/>
             <geometry>
-                <mesh filename="file:///ros2_ws/src/fastbot/fastbot_description/onshape/assets/n10_v2.stl"/>
+                <mesh filename="$(find-pkg-share fastbot_description)/onshape/assets/n10_v2.stl"/>
             </geometry>
         </collision>
@@ -232,5 +232,5 @@
             <origin xyz="-0.0105 0.0125 -0.00212" rpy="3.14159 -3.05067e-31 -1.55575e-61"/>
             <geometry>
-                <mesh filename="file:///ros2_ws/src/fastbot/fastbot_description/onshape/assets/part_33.stl"/>
+                <mesh filename="$(find-pkg-share fastbot_description)/onshape/assets/part_33.stl"/>
             </geometry>
             <material name="camera_material">
@@ -241,5 +241,5 @@
             <origin xyz="-0.0105 0.0125 -0.00212" rpy="3.14159 -3.05067e-31 -1.55575e-61"/>
             <geometry>
-                <mesh filename="file:///ros2_ws/src/fastbot/fastbot_description/onshape/assets/part_33.stl"/>
+                <mesh filename="$(find-pkg-share fastbot_description)/onshape/assets/part_33.stl"/>
             </geometry>
         </collision>
