Commit message: Update fastbot.xacro

File: fastbot/fastbot_description/models/urdf/fastbot.xacro (robot description, xacro)
@@ -4,33 +4,31 @@
 <robot name="fastbot" xmlns:xacro="http://ros.org/wiki/xacro">
   <xacro:property name="PI" value="3.141592653589793" />
-  <xacro:macro name="fastbot_body" params="robot_name">
-    <!-- Link base_link -->
-    <link name="${robot_name}_base_link">
-        <inertial>
-            <origin xyz="0 0 0" rpy="0 0 0"/>
+  <xacro:macro name="fastbot" params="robot_name">
+    <!-- Link fastbot_chassis -->
+    <link name="base_link">
+        <inertial>
+            <origin xyz="1.61253e-05 0.000669263 0.059916" rpy="0 0 0"/>
             <mass value="0.24695"/>
-            <inertia ixx="0.0007665739583333334" ixy="0.0" ixz="0.0" iyy="0.0005684994791666666" iyz="0.0" izz="0.0007907544791666667"/>
+            <inertia ixx="0.000946018" ixy="-8.62213e-08" ixz="-1.4272e-08" iyy="0.000732103" iyz="1.16569e-05" izz="0.000816741"/>
         </inertial>
         <!-- Part fastbot_chassis -->
         <visual>
-            <origin xyz="0.0573343 -0.0691426 0.00134516" rpy="0 -0 3.14159"/>
+            <origin xyz="0.06 -0.0698336 -0.002" rpy="0 -0 3.14159"/>
             <geometry>
                 <mesh filename="file:///ros2_ws/src/fastbot/fastbot_description/onshape/assets/fastbot_chassis.stl"/>
             </geometry>
-            <material name="fastbot_chassis_material">
+            <material name="base_link_material">
                 <color rgba="0.262745 0.282353 0.301961 1.0"/>
             </material>
         </visual>
         <collision>
-            <origin xyz="0.0573343 -0.0691426 0.00134516" rpy="0 -0 3.14159"/>
-            <!--<origin xyz="0.0 0.0 -0.00134516" rpy="0 0 0"/>-->
+            <origin xyz="0.06 -0.0698336 -0.002" rpy="0 -0 3.14159"/>
             <geometry>
                 <mesh filename="file:///ros2_ws/src/fastbot/fastbot_description/onshape/assets/fastbot_chassis.stl"/>
-                <!--<box size="0.12 0.155 0.115" />-->
-            </geometry>
-        </collision>
-    </link>
-    <!-- Link fastbot_motor -->
-    <link name="${robot_name}_motor_1">
+            </geometry>
+        </collision>
+    </link>
+    <!-- Link motor -->
+    <link name="motor">
         <inertial>
             <origin xyz="0.0067446 0.0085 -0.00855065" rpy="0 0 0"/>
@@ -56,11 +54,11 @@
     </link>
     <!-- Link wheel_right -->
-    <link name="${robot_name}_wheel_right">
-        <inertial>
-            <origin xyz="0 0 0" rpy="0 0 0"/>
-            <mass value="0.03"/>
-            <inertia ixx="1.0444293461874998e-05" ixy="0" ixz="0" iyy="1.0444293461874998e-05" iyz="0" izz="1.7812890903749995e-05"/>
-        </inertial>
-        <!-- Part wheel_d65x25_v1 -->
+    <link name="wheel_right">
+        <inertial>
+            <origin xyz="0 0 0" rpy="0 0 0"/>
+            <mass value="1e-09"/>
+            <inertia ixx="1e-09" ixy="0" ixz="0" iyy="1e-09" iyz="0" izz="1e-09"/>
+        </inertial>
+        <!-- Part wheel_right -->
         <visual>
             <origin xyz="0.1135 0.0162 0.103475" rpy="1.5708 1.5708 0"/>
@@ -68,5 +66,5 @@
                 <mesh filename="file:///ros2_ws/src/fastbot/fastbot_description/onshape/assets/wheel_d65x25_v1.stl"/>
             </geometry>
-            <material name="wheel_d65x25_v1_material">
+            <material name="wheel_right_material">
                 <color rgba="0.290196 0.290196 0.290196 1.0"/>
             </material>
@@ -78,37 +76,39 @@
             </geometry>
         </collision>
-        <!-- Part wheel_d65x25_v1_2 -->
-        <visual>
-            <origin xyz="0.1135 0.0162 0.1039" rpy="1.5708 1.5708 0"/>
-            <geometry>
-                <mesh filename="file:///ros2_ws/src/fastbot/fastbot_description/onshape/assets/wheel_d65x25_v1__2.stl"/>
-            </geometry>
-            <material name="wheel_d65x25_v1_2_material">
-                <color rgba="1 0.933333 0.133333 1.0"/>
-            </material>
-        </visual>
-        <collision>
-            <origin xyz="0.1135 0.0162 0.1039" rpy="1.5708 1.5708 0"/>
-            <geometry>
-                <mesh filename="file:///ros2_ws/src/fastbot/fastbot_description/onshape/assets/wheel_d65x25_v1__2.stl"/>
-            </geometry>
-        </collision>
-    </link>
-    <!-- Joint from fastbot_motor to wheel_d65x25_v1 -->
-    <joint name="${robot_name}_right_wheel" type="continuous">
-        <origin xyz="-0.02 0.0085 -0.0191" rpy="0 0 0"/>
-        <parent link="${robot_name}_motor_1"/>
-        <child link="${robot_name}_wheel_right"/>
-        <axis xyz="0 0 1"/>
-    </joint>
-    <!-- Joint from fastbot_chassis to fastbot_motor -->
-    <joint name="${robot_name}_right_motor" type="fixed">
-        <origin xyz="-0.0266657 0.0243574 0.0260952" rpy="-1.5708 -2.94692e-47 -1.5708"/>
-        <parent link="${robot_name}_base_link"/>
-        <child link="${robot_name}_motor_1"/>
-        <axis xyz="0 0 1"/>
-    </joint>
-    <!-- Link fastbot_motor_2 -->
-    <link name="${robot_name}_motor_2">
+        <!-- Part wheel_left -->
+        <visual>
+            <origin xyz="0.1135 0.0162 0.1039" rpy="1.5708 1.5708 0"/>
+            <geometry>
+                <mesh filename="file:///ros2_ws/src/fastbot/fastbot_description/onshape/assets/wheel_d65x25_v1__2.stl"/>
+            </geometry>
+            <material name="wheel_left_material">
+                <color rgba="0.290196 0.290196 0.290196 1.0"/>
+            </material>
+        </visual>
+        <collision>
+            <origin xyz="0.1135 0.0162 0.1039" rpy="1.5708 1.5708 0"/>
+            <geometry>
+                <mesh filename="file:///ros2_ws/src/fastbot/fastbot_description/onshape/assets/wheel_d65x25_v1__2.stl"/>
+            </geometry>
+        </collision>
+    </link>
+    <!-- Joint from motor to wheel_right -->
+    <joint name="right_wheel" type="continuous">
+        <origin xyz="-0.02 0.0085 -0.0191" rpy="4.35106e-30 2.46519e-32 3.14159"/>
+        <parent link="motor"/>
+        <child link="wheel_right"/>
+        <axis xyz="0 0 1"/>
+        <limit effort="10" velocity="10"/>
+    </joint>
+    <!-- Joint from base_link to motor -->
+    <joint name="right_motor" type="fixed">
+        <origin xyz="-0.024 0.0236664 0.02275" rpy="-1.5708 -2.94692e-47 -1.5708"/>
+        <parent link="base_link"/>
+        <child link="motor"/>
+        <axis xyz="0 0 1"/>
+        <limit effort="10" velocity="10"/>
+    </joint>
+    <!-- Link motor_2 -->
+    <link name="motor_2">
         <inertial>
             <origin xyz="0.0067446 -0.0085 -0.00855065" rpy="0 0 0"/>
@@ -133,10 +133,10 @@
         </collision>
     </link>
-    <!-- Link wheel_d65x25_v1_2 -->
-    <link name="${robot_name}_wheel_left">
-        <inertial>
-            <origin xyz="0 0 0" rpy="0 0 0"/>
-            <mass value="0.03"/>
-            <inertia ixx="1.0444293461874998e-05" ixy="0" ixz="0" iyy="1.0444293461874998e-05" iyz="0" izz="1.7812890903749995e-05"/>
+    <!-- Link wheel_left -->
+    <link name="wheel_left">
+        <inertial>
+            <origin xyz="0 0 0" rpy="0 0 0"/>
+            <mass value="1e-09"/>
+            <inertia ixx="1e-09" ixy="0" ixz="0" iyy="1e-09" iyz="0" izz="1e-09"/>
         </inertial>
         <!-- Part wheel_d65x25_v1_3 -->
@@ -147,5 +147,5 @@
             </geometry>
             <material name="wheel_d65x25_v1_3_material">
-                <color rgba="1 0.933333 0.133333 1.0"/>
+                <color rgba="0.290196 0.290196 0.290196 1.0"/>
             </material>
         </visual>
@@ -173,32 +173,34 @@
         </collision>
     </link>
-    <!-- Joint from fastbot_motor_2 to wheel_d65x25_v1_2 -->
-    <joint name="${robot_name}_left_wheel" type="continuous">
-        <origin xyz="-0.02 -0.0085 -0.0191" rpy="0 0 0"/>
-        <parent link="${robot_name}_motor_2"/>
-        <child link="${robot_name}_wheel_left"/>
-        <axis xyz="0 0 -1"/>
-    </joint>
-    <!-- Joint from fastbot_chassis to fastbot_motor_2 -->
-    <joint name="${robot_name}_left_motor" type="fixed">
-        <origin xyz="0.0213343 0.0243574 0.0260952" rpy="1.5708 -2.96391e-30 -1.5708"/>
-        <parent link="${robot_name}_base_link"/>
-        <child link="${robot_name}_motor_2"/>
-        <axis xyz="0 0 1"/>
-    </joint>
-    <!-- Link lslidar_n10 -->
-    <link name="${robot_name}_lidar">
-        <inertial>
-            <origin xyz="0 0 0" rpy="0 0 0"/>
-            <mass value="0.05"/>
-            <inertia ixx="0.0001" ixy="0" ixz="0" iyy="0.0001" iyz="0" izz="0.0002"/>
-        </inertial>
-        <!-- Part lslidar_n10 -->
+    <!-- Joint from motor_2 to wheel_left -->
+    <joint name="left_wheel" type="continuous">
+        <origin xyz="-0.02 -0.0085 -0.0191" rpy="-1.2326e-32 -1.54074e-33 3.14159"/>
+        <parent link="motor_2"/>
+        <child link="wheel_left"/>
+        <axis xyz="0 0 1"/>
+        <limit effort="10" velocity="10"/>
+    </joint>
+    <!-- Joint from base_link to motor_2 -->
+    <joint name="left_motor" type="fixed">
+        <origin xyz="0.024 0.0236664 0.02275" rpy="1.5708 -2.96391e-30 -1.5708"/>
+        <parent link="base_link"/>
+        <child link="motor_2"/>
+        <axis xyz="0 0 1"/>
+        <limit effort="10" velocity="10"/>
+    </joint>
+    <!-- Link n10_v2 -->
+    <link name="n10_v2">
+        <inertial>
+            <origin xyz="0 0 0" rpy="0 0 0"/>
+            <mass value="1e-09"/>
+            <inertia ixx="1e-09" ixy="0" ixz="0" iyy="1e-09" iyz="0" izz="1e-09"/>
+        </inertial>
+        <!-- Part n10_v2 -->
         <visual>
             <origin xyz="-0.074 -0.06 0.11" rpy="-3.14159 5.94511e-32 -8.90522e-65"/>
             <geometry>
-                <mesh filename="file:///ros2_ws/src/fastbot/fastbot_description/onshape/assets/lslidar_n10.stl"/>
-            </geometry>
-            <material name="lslidar_n10_material">
+                <mesh filename="file:///ros2_ws/src/fastbot/fastbot_description/onshape/assets/n10_v2.stl"/>
+            </geometry>
+            <material name="n10_v2_material">
                 <color rgba="0.0980392 0.0980392 0.0980392 1.0"/>
             </material>
@@ -207,29 +209,30 @@
             <origin xyz="-0.074 -0.06 0.11" rpy="-3.14159 5.94511e-32 -8.90522e-65"/>
             <geometry>
-                <mesh filename="file:///ros2_ws/src/fastbot/fastbot_description/onshape/assets/lslidar_n10.stl"/>
-            </geometry>
-        </collision>
-    </link>
-    <!-- Joint from fastbot_chassis to lslidar_n10 -->
-    <joint name="${robot_name}_lidar" type="fixed">
-        <origin xyz="-0.0166657 0 0.112" rpy="3.14159 1.13983e-46 -3.14159"/>
-        <parent link="${robot_name}_base_link"/>
-        <child link="${robot_name}_lidar"/>
-        <axis xyz="0 0 1"/>
-    </joint>
-    <!-- Link raspicam -->
-    <link name="${robot_name}_camera">
-        <inertial>
-            <origin xyz="0 0 0" rpy="0 0 0"/>
-            <mass value="0.01"/>
-            <inertia ixx="1e-09" ixy="0" ixz="0" iyy="1e-09" iyz="0" izz="1e-09"/>
-        </inertial>
-        <!-- Part raspicam -->
+                <mesh filename="file:///ros2_ws/src/fastbot/fastbot_description/onshape/assets/n10_v2.stl"/>
+            </geometry>
+        </collision>
+    </link>
+    <!-- Joint from base_link to n10_v2 -->
+    <joint name="lidar" type="fixed">
+        <origin xyz="-0.014 -0.00983363 0.108" rpy="3.14159 1.13983e-46 -3.14159"/>
+        <parent link="base_link"/>
+        <child link="n10_v2"/>
+        <axis xyz="0 0 1"/>
+        <limit effort="10" velocity="10"/>
+    </joint>
+    <!-- Link camera -->
+    <link name="camera">
+        <inertial>
+            <origin xyz="0 0 0" rpy="0 0 0"/>
+            <mass value="1e-09"/>
+            <inertia ixx="1e-09" ixy="0" ixz="0" iyy="1e-09" iyz="0" izz="1e-09"/>
+        </inertial>
+        <!-- Part camera -->
         <visual>
             <origin xyz="-0.0105 0.0125 -0.00212" rpy="3.14159 -3.05067e-31 -1.55575e-61"/>
             <geometry>
-                <mesh filename="file:///ros2_ws/src/fastbot/fastbot_description/onshape/assets/raspicam.stl"/>
-            </geometry>
-            <material name="raspicam_material">
+                <mesh filename="file:///ros2_ws/src/fastbot/fastbot_description/onshape/assets/part_33.stl"/>
+            </geometry>
+            <material name="camera_material">
                 <color rgba="0.34902 0.376471 0.4 1.0"/>
             </material>
@@ -238,44 +241,15 @@
             <origin xyz="-0.0105 0.0125 -0.00212" rpy="3.14159 -3.05067e-31 -1.55575e-61"/>
             <geometry>
-                <mesh filename="file:///ros2_ws/src/fastbot/fastbot_description/onshape/assets/raspicam.stl"/>
-            </geometry>
-        </collision>
-    </link>
-    <!-- Joint from fastbot_chassis to raspicam -->
-    <joint name="${robot_name}_camera" type="fixed">
-        <origin xyz="0.00783428 -0.0661426 0.100995" rpy="0 0 -1.5708"/>
-        <parent link="${robot_name}_base_link"/>
-        <child link="${robot_name}_camera"/>
-        <axis xyz="0 0 1"/>
-    </joint>
-    <!-- Link pololu_ball_caster -->
-    <link name="${robot_name}_ball_caster">
-        <inertial>
-            <origin xyz="0 0 0" rpy="0 0 0"/>
-            <mass value="0.01"/>
-            <inertia ixx="1e-09" ixy="0" ixz="0" iyy="1e-09" iyz="0" izz="1e-09"/>
-        </inertial>
-        <visual>
-            <origin xyz="0.006731 0 -0.0106945" rpy="-1.5708 -0 0"/>
-            <geometry>
-                <mesh filename="file:///ros2_ws/src/fastbot/fastbot_description/onshape/assets/pololu_ball_caster.stl"/>
-            </geometry>
-            <material name="pololu_ball_caster_material">
-                <color rgba="0.34902 0.376471 0.4 1.0"/>
-            </material>
-        </visual>
-        <collision>
-            <origin xyz="0.006731 0 -0.0106945" rpy="-1.5708 -0 0"/>
-            <geometry>
-                <mesh filename="file:///ros2_ws/src/fastbot/fastbot_description/onshape/assets/pololu_ball_caster.stl"/>
-            </geometry>
-        </collision>
-    </link>
-    <!-- Joint from fastbot_chassis to pololu_ball_caster -->
-    <joint name="caster" type="fixed">
-        <origin xyz="-0.0100317 -0.0541426 0.00334516" rpy="0 -0 0"/>
-        <parent link="${robot_name}_base_link"/>
-        <child link="${robot_name}_ball_caster"/>
-        <axis xyz="0 0 1"/>
+                <mesh filename="file:///ros2_ws/src/fastbot/fastbot_description/onshape/assets/part_33.stl"/>
+            </geometry>
+        </collision>
+    </link>
+    <!-- Joint from base_link to camera -->
+    <joint name="camera" type="fixed">
+        <origin xyz="0.0105 -0.0668336 0.09765" rpy="-1.5708 1.14468e-45 6.41848e-15"/>
+        <parent link="base_link"/>
+        <child link="camera"/>
+        <axis xyz="0 0 1"/>
+        <limit effort="10" velocity="10"/>
     </joint>
   </xacro:macro>

Commit message: Update fastbot.xacro

File: fastbot/fastbot_description/models/urdf/fastbot.xacro (robot description, xacro)
@@ -16,5 +16,5 @@
             <origin xyz="0.06 -0.0698336 -0.002" rpy="0 -0 3.14159"/>
             <geometry>
-                <mesh filename="file:///ros2_ws/src/fastbot/fastbot_description/onshape/assets/fastbot_chassis.stl"/>
+                <mesh filename="/root/ros2_ws/src/fastbot/fastbot_description/onshape/assets/fastbot_chassis.stl"/>
             </geometry>
             <material name="base_link_material">
@@ -25,5 +25,5 @@
             <origin xyz="0.06 -0.0698336 -0.002" rpy="0 -0 3.14159"/>
             <geometry>
-                <mesh filename="file:///ros2_ws/src/fastbot/fastbot_description/onshape/assets/fastbot_chassis.stl"/>
+                <mesh filename="/root/ros2_ws/src/fastbot/fastbot_description/onshape/assets/fastbot_chassis.stl"/>
             </geometry>
         </collision>
@@ -40,5 +40,5 @@
             <origin xyz="0.0935 -0.00775 -0.036" rpy="-1.5708 -1.5708 0"/>
             <geometry>
-                <mesh filename="file:///ros2_ws/src/fastbot/fastbot_description/onshape/assets/fastbot_motor.stl"/>
+                <mesh filename="/root/ros2_ws/src/fastbot/fastbot_description/onshape/assets/fastbot_motor.stl"/>
             </geometry>
             <material name="fastbot_motor_material">
@@ -49,5 +49,5 @@
             <origin xyz="0.0935 -0.00775 -0.036" rpy="-1.5708 -1.5708 0"/>
             <geometry>
-                <mesh filename="file:///ros2_ws/src/fastbot/fastbot_description/onshape/assets/fastbot_motor.stl"/>
+                <mesh filename="/root/ros2_ws/src/fastbot/fastbot_description/onshape/assets/fastbot_motor.stl"/>
             </geometry>
         </collision>
@@ -64,5 +64,5 @@
             <origin xyz="0.1135 0.0162 0.103475" rpy="1.5708 1.5708 0"/>
             <geometry>
-                <mesh filename="file:///ros2_ws/src/fastbot/fastbot_description/onshape/assets/wheel_d65x25_v1.stl"/>
+                <mesh filename="/root/ros2_ws/src/fastbot/fastbot_description/onshape/assets/wheel_d65x25_v1.stl"/>
             </geometry>
             <material name="wheel_right_material">
@@ -73,5 +73,5 @@
             <origin xyz="0.1135 0.0162 0.103475" rpy="1.5708 1.5708 0"/>
             <geometry>
-                <mesh filename="file:///ros2_ws/src/fastbot/fastbot_description/onshape/assets/wheel_d65x25_v1.stl"/>
+                <mesh filename="/root/ros2_ws/src/fastbot/fastbot_description/onshape/assets/wheel_d65x25_v1.stl"/>
             </geometry>
         </collision>
@@ -80,5 +80,5 @@
             <origin xyz="0.1135 0.0162 0.1039" rpy="1.5708 1.5708 0"/>
             <geometry>
-                <mesh filename="file:///ros2_ws/src/fastbot/fastbot_description/onshape/assets/wheel_d65x25_v1__2.stl"/>
+                <mesh filename="/root/ros2_ws/src/fastbot/fastbot_description/onshape/assets/wheel_d65x25_v1__2.stl"/>
             </geometry>
             <material name="wheel_left_material">
@@ -89,5 +89,5 @@
             <origin xyz="0.1135 0.0162 0.1039" rpy="1.5708 1.5708 0"/>
             <geometry>
-                <mesh filename="file:///ros2_ws/src/fastbot/fastbot_description/onshape/assets/wheel_d65x25_v1__2.stl"/>
+                <mesh filename="/root/ros2_ws/src/fastbot/fastbot_description/onshape/assets/wheel_d65x25_v1__2.stl"/>
             </geometry>
         </collision>
@@ -120,5 +120,5 @@
             <origin xyz="0.0935 -0.02475 -0.036" rpy="-1.5708 -1.5708 0"/>
             <geometry>
-                <mesh filename="file:///ros2_ws/src/fastbot/fastbot_description/onshape/assets/fastbot_motor.stl"/>
+                <mesh filename="/root/ros2_ws/src/fastbot/fastbot_description/onshape/assets/fastbot_motor.stl"/>
             </geometry>
             <material name="fastbot_motor_2_material">
@@ -129,5 +129,5 @@
             <origin xyz="0.0935 -0.02475 -0.036" rpy="-1.5708 -1.5708 0"/>
             <geometry>
-                <mesh filename="file:///ros2_ws/src/fastbot/fastbot_description/onshape/assets/fastbot_motor.stl"/>
+                <mesh filename="/root/ros2_ws/src/fastbot/fastbot_description/onshape/assets/fastbot_motor.stl"/>
             </geometry>
         </collision>
@@ -144,5 +144,5 @@
             <origin xyz="0.1135 0.0162 0.1039" rpy="1.5708 1.5708 0"/>
             <geometry>
-                <mesh filename="file:///ros2_ws/src/fastbot/fastbot_description/onshape/assets/wheel_d65x25_v1__2.stl"/>
+                <mesh filename="/root/ros2_ws/src/fastbot/fastbot_description/onshape/assets/wheel_d65x25_v1__2.stl"/>
             </geometry>
             <material name="wheel_d65x25_v1_3_material">
@@ -153,5 +153,5 @@
             <origin xyz="0.1135 0.0162 0.1039" rpy="1.5708 1.5708 0"/>
             <geometry>
-                <mesh filename="file:///ros2_ws/src/fastbot/fastbot_description/onshape/assets/wheel_d65x25_v1__2.stl"/>
+                <mesh filename="/root/ros2_ws/src/fastbot/fastbot_description/onshape/assets/wheel_d65x25_v1__2.stl"/>
             </geometry>
         </collision>
@@ -160,5 +160,5 @@
             <origin xyz="0.1135 0.0162 0.104325" rpy="1.5708 1.5708 0"/>
             <geometry>
-                <mesh filename="file:///ros2_ws/src/fastbot/fastbot_description/onshape/assets/wheel_d65x25_v1.stl"/>
+                <mesh filename="/root/ros2_ws/src/fastbot/fastbot_description/onshape/assets/wheel_d65x25_v1.stl"/>
             </geometry>
             <material name="wheel_d65x25_v1_4_material">
@@ -169,5 +169,5 @@
             <origin xyz="0.1135 0.0162 0.104325" rpy="1.5708 1.5708 0"/>
             <geometry>
-                <mesh filename="file:///ros2_ws/src/fastbot/fastbot_description/onshape/assets/wheel_d65x25_v1.stl"/>
+                <mesh filename="/root/ros2_ws/src/fastbot/fastbot_description/onshape/assets/wheel_d65x25_v1.stl"/>
             </geometry>
         </collision>
@@ -200,5 +200,5 @@
             <origin xyz="-0.074 -0.06 0.11" rpy="-3.14159 5.94511e-32 -8.90522e-65"/>
             <geometry>
-                <mesh filename="file:///ros2_ws/src/fastbot/fastbot_description/onshape/assets/n10_v2.stl"/>
+                <mesh filename="/root/ros2_ws/src/fastbot/fastbot_description/onshape/assets/n10_v2.stl"/>
             </geometry>
             <material name="n10_v2_material">
@@ -209,5 +209,5 @@
             <origin xyz="-0.074 -0.06 0.11" rpy="-3.14159 5.94511e-32 -8.90522e-65"/>
             <geometry>
-                <mesh filename="file:///ros2_ws/src/fastbot/fastbot_description/onshape/assets/n10_v2.stl"/>
+                <mesh filename="/root/ros2_ws/src/fastbot/fastbot_description/onshape/assets/n10_v2.stl"/>
             </geometry>
         </collision>
@@ -232,5 +232,5 @@
             <origin xyz="-0.0105 0.0125 -0.00212" rpy="3.14159 -3.05067e-31 -1.55575e-61"/>
             <geometry>
-                <mesh filename="file:///ros2_ws/src/fastbot/fastbot_description/onshape/assets/part_33.stl"/>
+                <mesh filename="/root/ros2_ws/src/fastbot/fastbot_description/onshape/assets/part_33.stl"/>
             </geometry>
             <material name="camera_material">
@@ -241,5 +241,5 @@
             <origin xyz="-0.0105 0.0125 -0.00212" rpy="3.14159 -3.05067e-31 -1.55575e-61"/>
             <geometry>
-                <mesh filename="file:///ros2_ws/src/fastbot/fastbot_description/onshape/assets/part_33.stl"/>
+                <mesh filename="/root/ros2_ws/src/fastbot/fastbot_description/onshape/assets/part_33.stl"/>
             </geometry>
         </collision>
